File: kicad/320_SDCARD.sch (KiCad schematic (older format))
At the start: 3 parts, among them J320 Micro_SD_Card_Det, U101 74LS07

Commit message: ran autoroute
Parts:
- RN320: value R_Network05 -> 10k
Changed lines of the file:
@@
 P 5450 2950
 F 0 "RN320" H 5738 2996 50  0000 L CNN
-F 1 "R_Network05" H 5738 2905 50  0000 L CNN
+F 1 "10k" H 5738 2905 50  0000 L CNN
 F 2 "Resistor_THT:R_Array_SIP6" V 5825 2950 50  0001 C CNN
 F 3 "http://www.vishay.com/docs/31509/csc.pdf" H 5450 2950 50  0001 C CNN
