File: kicad/_autosave-68k8.kicad_pcb (KiCad board)
At the start: 2 copper layers, 160 x 114.3 mm, 57 parts, among them J0 Barrel_Jack, J300 Conn_01x02_Male, J301 Conn_01x03_Male, J302 USB_B, J303 Conn_01x07, J320 Micro_SD_Card_Det, J330 Conn_02x04_Top_Bottom, SW110 SW_Push, U1 LF33_TO220, U100 68008D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

Commit message: ran autoroute
Routing:
- net (no net): track 22.5 -> 0.00 mm
- net +5V: track 213.9 -> 236.4 mm
Changed lines of the file:
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@@
   (general
     (thickness 1.6)
-    (drawings 5)
+    (drawings 7)
     (tracks 1569)
     (zones 0)
@@
     (pcbplotparams
       (layerselection 0x010fc_ffffffff)
-      (usegerberextensions false)
-      (usegerberattributes true)
-      (usegerberadvancedattributes true)
-      (creategerberjobfile true)
+      (usegerberextensions true)
+      (usegerberattributes false)
+      (usegerberadvancedattributes false)
+      (creategerberjobfile false)
       (excludeedgelayer true)
       (linewidth 0.100000)
@@
       (plotinvisibletext false)
       (padsonsilk false)
-      (subtractmaskfromsilk false)
+      (subtractmaskfromsilk true)
       (outputformat 1)
       (mirror false)
-      (drillshape 1)
+      (drillshape 0)
       (scaleselection 1)
-      (outputdirectory ""))
+      (outputdirectory "Gerber/"))
   )
   (net 0 "")
@@
     )
   )
+  (dimension 160.02 (width 0.15) (layer Cmts.User)
+    (gr_text "160.020 mm" (at 212.09 -5.11) (layer Cmts.User)
+      (effects (font (size 1 1) (thickness 0.15)))
+    )
+    (feature1 (pts (xy 292.1 10.16) (xy 292.1 -4.396421)))
+    (feature2 (pts (xy 132.08 10.16) (xy 132.08 -4.396421)))
+    (crossbar (pts (xy 132.08 -3.81) (xy 292.1 -3.81)))
+    (arrow1a (pts (xy 292.1 -3.81) (xy 290.973496 -3.223579)))
+    (arrow1b (pts (xy 292.1 -3.81) (xy 290.973496 -4.396421)))
+    (arrow2a (pts (xy 132.08 -3.81) (xy 133.206504 -3.223579)))
+    (arrow2b (pts (xy 132.08 -3.81) (xy 133.206504 -4.396421)))
+  )
+  (dimension 114.3 (width 0.15) (layer Cmts.User)
+    (gr_text "114.300 mm" (at 320.07 67.31 270) (layer Cmts.User)
+      (effects (font (size 1 1) (thickness 0.15)))
+    )
+    (feature1 (pts (xy 292.1 124.46) (xy 319.356421 124.46)))
+    (feature2 (pts (xy 292.1 10.16) (xy 319.356421 10.16)))
+    (crossbar (pts (xy 318.77 10.16) (xy 318.77 124.46)))
+    (arrow1a (pts (xy 318.77 124.46) (xy 318.183579 123.333496)))
+    (arrow1b (pts (xy 318.77 124.46) (xy 319.356421 123.333496)))
+    (arrow2a (pts (xy 318.77 10.16) (xy 318.183579 11.286504)))
+    (arrow2b (pts (xy 318.77 10.16) (xy 319.356421 11.286504)))
+  )
   (gr_line (start 292.1 10.16) (end 292.1 124.46) (layer Edge.Cuts) (width 0.1))
   (gr_line (start 132.08 10.16) (end 292.1 10.16) (layer Edge.Cuts) (width 0.1))
@@
     (arrow2b (pts (xy 283.972 61.214) (xy 284.558421 62.340504)))
   )
-  (via (at 144.903053 78.616947) (size 0.8) (drill 0.4) (layers F.Cu B.Cu) (net 6))
-  (segment (start 152.501107 86.215001) (end 162.704999 86.215001) (width 0.25) (layer F.Cu) (net 0))
-  (segment (start 144.903053 78.616947) (end 152.501107 86.215001) (width 0.25) (layer F.Cu) (net 0))
-  (via (at 163.83 85.09) (size 0.8) (drill 0.4) (layers F.Cu B.Cu) (net 6))
-  (segment (start 162.704999 86.215001) (end 163.83 85.09) (width 0.25) (layer F.Cu) (net 0))
+  (segment (start 153.67 85.09) (end 153.67 53.34) (width 0.25) (layer B.Cu) (net 1))
+  (segment (start 153.67 53.34) (end 158.75 48.26) (width 0.25) (layer B.Cu) (net 1))
+  (segment (start 158.75 85.09) (end 153.67 85.09) (width 0.25) (layer F.Cu) (net 1))
   (segment (start 180.271792 63.431792) (end 182.743584 60.96) (width 0.25) (layer B.Cu) (net 2))
   (segment (start 182.743584 60.96) (end 189.23 60.96) (width 0.25) (layer B.Cu) (net 2))
@@
   (segment (start 149.86 88.9) (end 148.59 87.63) (width 0.25) (layer B.Cu) (net 2))
   (via (at 138.43 95.25) (size 0.8) (drill 0.4) (layers F.Cu B.Cu) (net 2))
-  (via (at 158.75 25.4) (size 0.8) (drill 0.4) (layers F.Cu B.Cu) (net 6))
-  (segment (start 153.67 85.09) (end 153.67 53.34) (width 0.25) (layer B.Cu) (net 1))
-  (segment (start 153.67 53.34) (end 158.75 48.26) (width 0.25) (layer B.Cu) (net 1))
-  (segment (start 158.75 85.09) (end 153.67 85.09) (width 0.25) (layer F.Cu) (net 1))
   (segment (start 203.2 50.8) (end 210.82 50.8) (width 0.25) (layer F.Cu) (net 2))
   (segment (start 203.2 86.36) (end 210.82 86.36) (width 0.25) (layer F.Cu) (net 2))
@@
   (segment (start 147.32 109.22) (end 160.02 109.22) (width 0.25) (layer F.Cu) (net 5))
   (via (at 160.02 109.22) (size 0.8) (drill 0.4) (layers F.Cu B.Cu) (net 5))
+  (segment (start 152.501107 86.215001) (end 162.704999 86.215001) (width 0.25) (layer F.Cu) (net 6))
+  (segment (start 144.903053 78.616947) (end 152.501107 86.215001) (width 0.25) (layer F.Cu) (net 6))
+  (segment (start 162.704999 86.215001) (end 163.83 85.09) (width 0.25) (layer F.Cu) (net 6))
+  (via (at 144.903053 78.616947) (size 0.8) (drill 0.4) (layers F.Cu B.Cu) (net 6))
+  (via (at 163.83 85.09) (size 0.8) (drill 0.4) (layers F.Cu B.Cu) (net 6))
+  (via (at 158.75 25.4) (size 0.8) (drill 0.4) (layers F.Cu B.Cu) (net 6))
   (segment (start 162.56 104.14) (end 162.56 103.0147) (width 0.25) (layer B.Cu) (net 6))
   (segment (start 161.29 89.1436) (end 161.29 101.7447) (width 0.25) (layer B.Cu) (net 6))
