File: kicad/68k8.kicad_pcb (KiCad board)
At the start: 2 copper layers, 160 x 114.3 mm, 57 parts, among them J0 Barrel_Jack, J300 Conn_01x02_Male, J301 Conn_01x03_Male, J302 USB_B, J303 Conn_01x07, J320 Micro_SD_Card_Det, J330 Conn_02x04_Top_Bottom, SW110 SW_Push, U1 LF33_TO220, U100 68008D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

Commit message: key routes placed
Parts:
- moved C330 1.80 mm to (170.2, 92.7)
- moved C331 1.80 mm to (161.3, 92.7)
Routing:
- net DART_RX: track 0.00 -> 148.6 mm, vias 0 -> 1
- net DART_TX: track 0.00 -> 142.7 mm, vias 0 -> 1
- net SCLK: track 0.00 -> 50.6 mm, vias 0 -> 1
- net MOSI: track 0.00 -> 40.7 mm, vias 0 -> 1
- net PROG_EN: track 47.1 -> 25.8 mm, vias 1 -> 0
- net PROG_SCLK: track 10.8 -> 21.9 mm, vias 0 -> 1
- net MISO: track 79.1 -> 81.3 mm, vias 1 -> 2
Changed lines of the file:
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@@
     (thickness 1.6)
     (drawings 6)
-    (tracks 113)
+    (tracks 155)
     (zones 0)
     (modules 57)
@@
   )
   (module Capacitor_THT:C_Rect_L4.0mm_W2.5mm_P2.50mm (layer F.Cu)
-    (at 168.91 93.98 180)
+    (at 170.18 92.71 180)
     (descr "C, Rect series, Radial, pin pitch=2.50mm, , length*width=4*2.5mm^2, Capacitor")
     (tags "C Rect series Radial pin pitch 2.50mm  length 4mm width 2.5mm Capacitor")
@@
   )
   (module Capacitor_THT:C_Rect_L4.0mm_W2.5mm_P2.50mm (layer F.Cu)
-    (at 160.02 93.98 180)
+    (at 161.29 92.71 180)
     (descr "C, Rect series, Radial, pin pitch=2.50mm, , length*width=4*2.5mm^2, Capacitor")
     (tags "C Rect series Radial pin pitch 2.50mm  length 4mm width 2.5mm Capacitor")
@@
   (via (at 265.43 100.33) (size 0.8) (drill 0.4) (layers F.Cu B.Cu) (net 17))
   (segment (start 265.43 110.32) (end 265.43 100.33) (width 0.25) (layer B.Cu) (net 17))
-  (segment (start 248.92 100.33) (end 245.11 96.52) (width 0.25) (layer F.Cu) (net 17))
-  (segment (start 265.43 100.33) (end 248.92 100.33) (width 0.25) (layer F.Cu) (net 17))
+  (segment (start 265.43 100.33) (end 250.82359 100.33) (width 0.25) (layer F.Cu) (net 17))
+  (segment (start 250.82359 100.33) (end 249.55359 99.06) (width 0.25) (layer F.Cu) (net 17))
+  (segment (start 247.65 99.06) (end 245.11 96.52) (width 0.25) (layer F.Cu) (net 17))
+  (segment (start 249.55359 99.06) (end 247.65 99.06) (width 0.25) (layer F.Cu) (net 17))
+  (segment (start 146.194999 103.079999) (end 147.674998 101.6) (width 0.25) (layer F.Cu) (net 18))
+  (segment (start 146.194999 105.554999) (end 146.194999 103.079999) (width 0.25) (layer F.Cu) (net 18))
+  (segment (start 147.32 106.68) (end 146.194999 105.554999) (width 0.25) (layer F.Cu) (net 18))
+  (segment (start 147.674998 101.6) (end 177.8 101.6) (width 0.25) (layer F.Cu) (net 18))
+  (via (at 179.07 102.87) (size 0.8) (drill 0.4) (layers F.Cu B.Cu) (net 18))
+  (segment (start 177.8 101.6) (end 179.07 102.87) (width 0.25) (layer F.Cu) (net 18))
+  (segment (start 179.07 111.76) (end 181.61 114.3) (width 0.25) (layer B.Cu) (net 18))
+  (segment (start 179.07 102.87) (end 179.07 111.76) (width 0.25) (layer B.Cu) (net 18))
+  (segment (start 179.944998 114.3) (end 181.214998 113.03) (width 0.25) (layer F.Cu) (net 19))
+  (segment (start 161.991509 114.3) (end 179.944998 114.3) (width 0.25) (layer F.Cu) (net 19))
+  (segment (start 159.451509 116.84) (end 161.991509 114.3) (width 0.25) (layer F.Cu) (net 19))
+  (segment (start 154.94 116.84) (end 159.451509 116.84) (width 0.25) (layer F.Cu) (net 19))
+  (segment (start 181.214998 113.03) (end 186.69 113.03) (width 0.25) (layer F.Cu) (net 19))
+  (via (at 186.69 113.03) (size 0.8) (drill 0.4) (layers F.Cu B.Cu) (net 19))
+  (segment (start 186.69 109.22) (end 189.23 106.68) (width 0.25) (layer B.Cu) (net 19))
+  (segment (start 186.69 113.03) (end 186.69 109.22) (width 0.25) (layer B.Cu) (net 19))
   (segment (start 177.944999 118.254999) (end 175.26 115.57) (width 0.25) (layer F.Cu) (net 20))
   (segment (start 188.104999 118.254999) (end 177.944999 118.254999) (width 0.25) (layer F.Cu) (net 20))
   (segment (start 189.23 119.38) (end 188.104999 118.254999) (width 0.25) (layer F.Cu) (net 20))
-  (segment (start 147.32 116.84) (end 148.495001 118.015001) (width 0.25) (layer F.Cu) (net 20))
   (segment (start 146.18863 116.84) (end 147.32 116.84) (width 0.25) (layer B.Cu) (net 20))
   (segment (start 144.78 116.84) (end 146.18863 116.84) (width 0.25) (layer B.Cu) (net 20))
@@
   (segment (start 134.62 102.87) (end 134.62 106.68) (width 0.25) (layer B.Cu) (net 20))
   (segment (start 139.7 97.79) (end 134.62 102.87) (width 0.25) (layer B.Cu) (net 20))
-  (segment (start 148.495001 118.015001) (end 152.4 121.92) (width 0.25) (layer F.Cu) (net 20))
   (segment (start 152.4 121.92) (end 168.91 121.92) (width 0.25) (layer F.Cu) (net 20))
   (segment (start 168.91 121.92) (end 173.99 121.92) (width 0.25) (layer F.Cu) (net 20))
@@
   (segment (start 173.99 116.84) (end 175.26 115.57) (width 0.25) (layer B.Cu) (net 20))
   (segment (start 173.99 121.92) (end 173.99 116.84) (width 0.25) (layer B.Cu) (net 20))
+  (segment (start 147.32 116.84) (end 148.59 118.11) (width 0.25) (layer B.Cu) (net 20))
+  (segment (start 148.59 118.11) (end 148.59 121.92) (width 0.25) (layer B.Cu) (net 20))
+  (via (at 148.59 121.92) (size 0.8) (drill 0.4) (layers F.Cu B.Cu) (net 20))
+  (segment (start 152.4 121.92) (end 148.59 121.92) (width 0.25) (layer F.Cu) (net 20))
   (segment (start 195.58 108.055) (end 195.58 107.95) (width 0.25) (layer F.Cu) (net 27))
   (segment (start 209.015 121.49) (end 195.58 108.055) (width 0.25) (layer F.Cu) (net 27))
@@
   (segment (start 146.194999 105.265001) (end 146.194999 110.634999) (width 0.25) (layer B.Cu) (net 31))
   (segment (start 147.32 104.14) (end 146.194999 105.265001) (width 0.25) (layer B.Cu) (net 31))
-  (segment (start 175.26 110.49) (end 176.53 111.76) (width 0.25) (layer B.Cu) (net 31))
-  (segment (start 176.53 111.76) (end 176.53 120.65) (width 0.25) (layer B.Cu) (net 31))
-  (via (at 176.53 120.65) (size 0.8) (drill 0.4) (layers F.Cu B.Cu) (net 31))
-  (segment (start 167.64 120.65) (end 166.37 119.38) (width 0.25) (layer F.Cu) (net 31))
-  (segment (start 176.53 120.65) (end 167.64 120.65) (width 0.25) (layer F.Cu) (net 31))
-  (segment (start 161.29 113.03) (end 168.91 105.41) (width 0.25) (layer F.Cu) (net 32))
+  (segment (start 160.087919 116.84) (end 158.817919 118.11) (width 0.25) (layer F.Cu) (net 32))
+  (segment (start 161.29 116.84) (end 160.087919 116.84) (width 0.25) (layer F.Cu) (net 32))
+  (segment (start 158.817919 118.11) (end 149.86 118.11) (width 0.25) (layer F.Cu) (net 32))
+  (via (at 149.86 118.11) (size 0.8) (drill 0.4) (layers F.Cu B.Cu) (net 32))
+  (segment (start 149.86 111.76) (end 147.32 109.22) (width 0.25) (layer B.Cu) (net 32))
+  (segment (start 149.86 118.11) (end 149.86 111.76) (width 0.25) (layer B.Cu) (net 32))
   (segment (start 167.545001 118.204999) (end 168.91 116.84) (width 0.25) (layer F.Cu) (net 33))
-  (segment (start 156.115001 118.204999) (end 167.545001 118.204999) (width 0.25) (layer F.Cu) (net 33))
-  (segment (start 154.94 119.38) (end 156.115001 118.204999) (width 0.25) (layer F.Cu) (net 33))
   (segment (start 168.91 116.84) (end 168.91 111.76) (width 0.25) (layer B.Cu) (net 33))
+  (segment (start 159.004998 119.38) (end 154.94 119.38) (width 0.25) (layer F.Cu) (net 33))
+  (segment (start 160.179999 118.204999) (end 159.004998 119.38) (width 0.25) (layer F.Cu) (net 33))
+  (segment (start 167.545001 118.204999) (end 160.179999 118.204999) (width 0.25) (layer F.Cu) (net 33))
   (segment (start 148.445001 115.425001) (end 158.605001 115.425001) (width 0.25) (layer F.Cu) (net 34))
   (segment (start 147.32 114.3) (end 148.445001 115.425001) (width 0.25) (layer F.Cu) (net 34))
@@
   (segment (start 163.83 112.634998) (end 161.29 110.094998) (width 0.25) (layer B.Cu) (net 35))
   (segment (start 163.83 116.84) (end 163.83 112.634998) (width 0.25) (layer B.Cu) (net 35))
+  (segment (start 249.725001 101.135001) (end 231.945001 101.135001) (width 0.25) (layer F.Cu) (net 103))
+  (segment (start 252.73 104.14) (end 249.725001 101.135001) (width 0.25) (layer F.Cu) (net 103))
+  (segment (start 231.945001 101.135001) (end 227.474999 96.664999) (width 0.25) (layer F.Cu) (net 103))
+  (via (at 157.48 96.52) (size 0.8) (drill 0.4) (layers F.Cu B.Cu) (net 103))
+  (segment (start 157.335001 96.664999) (end 157.48 96.52) (width 0.25) (layer F.Cu) (net 103))
+  (segment (start 227.474999 96.664999) (end 157.335001 96.664999) (width 0.25) (layer F.Cu) (net 103))
+  (segment (start 157.48 96.52) (end 157.080001 96.120001) (width 0.25) (layer B.Cu) (net 103))
+  (segment (start 157.080001 55.009999) (end 157.48 54.61) (width 0.25) (layer B.Cu) (net 103))
+  (segment (start 157.080001 96.120001) (end 157.080001 55.009999) (width 0.25) (layer B.Cu) (net 103))
+  (segment (start 157.48 54.61) (end 158.75 53.34) (width 0.25) (layer B.Cu) (net 103))
+  (segment (start 250.006419 100.780009) (end 249.55641 100.33) (width 0.25) (layer F.Cu) (net 104))
+  (segment (start 251.910009 100.780009) (end 250.006419 100.780009) (width 0.25) (layer F.Cu) (net 104))
+  (segment (start 255.27 104.14) (end 251.910009 100.780009) (width 0.25) (layer F.Cu) (net 104))
+  (segment (start 249.55641 100.33) (end 232.41 100.33) (width 0.25) (layer F.Cu) (net 104))
+  (segment (start 232.41 100.33) (end 227.33 95.25) (width 0.25) (layer F.Cu) (net 104))
+  (segment (start 227.33 95.25) (end 157.124998 95.25) (width 0.25) (layer F.Cu) (net 104))
+  (segment (start 157.124998 95.25) (end 156.21 95.25) (width 0.25) (layer F.Cu) (net 104))
+  (via (at 156.21 95.25) (size 0.8) (drill 0.4) (layers F.Cu B.Cu) (net 104))
+  (segment (start 155.759991 53.790009) (end 158.75 50.8) (width 0.25) (layer B.Cu) (net 104))
+  (segment (start 155.759991 94.799991) (end 155.759991 53.790009) (width 0.25) (layer B.Cu) (net 104))
+  (segment (start 156.21 95.25) (end 155.759991 94.799991) (width 0.25) (layer B.Cu) (net 104))
   (zone (net 2) (net_name GND) (layer F.Cu) (hatch edge 0.508)
     (connect_pads (clearance 0.508))

Commit message: redid power routes
Parts:
- moved J300 47.8 mm to (137.4, 50.8), turned to 0 degrees
Routing:
- net +5V: track 8.15 -> 100.3 mm
- net GND: track 0.00 -> 47.7 mm
- net Net-(J300-Pad2): track 0.00 -> 6.10 mm
- net Net-(J300-Pad1): track 0.00 -> 6.10 mm

Commit message: almost done, almost
Parts:
- removed J0: Barrel_Jack, Connector_BarrelJack:BarrelJack_Horizontal
- added D0: POW_LED, LED_THT:LED_D3.0mm, F.Cu at (280.4, 71.6)
- added J00: Barrel_Jack_Switch, Connector_BarrelJack:BarrelJack_Horizontal, F.Cu at (243.8, 112.3)
- added R0: 2K, Resistor_THT:R_Axial_DIN0309_L9.0mm_D3.2mm_P2.54mm_Vertical, F.Cu at (272.0, 71.6)
- added REF**: KiCad-Logo2_5mm_SilkScreen, Symbol:KiCad-Logo2_5mm_SilkScreen, B.Cu at (195.3, 15.0)
- added REF**: OSHW-Symbol_6.7x6mm_SilkScreen, Symbol:OSHW-Symbol_6.7x6mm_SilkScreen, B.Cu at (262.6, 14.7)
Routing:
- net 555_01: track 6.35 -> 204.4 mm
- net RESET_IN: track 37.9 -> 223.2 mm
- net /100_CPU/A8: track 0.00 -> 184.9 mm, vias 0 -> 2
- net /100_CPU/A14: track 0.00 -> 174.1 mm, vias 0 -> 3
- net GND: track 47.7 -> 219.2 mm, vias 0 -> 9
- net /100_CPU/D3: track 0.00 -> 164.7 mm, vias 0 -> 1
- net /100_CPU/A6: track 0.00 -> 164.5 mm, vias 0 -> 2
- net /100_CPU/A12: track 0.00 -> 162.8 mm, vias 0 -> 3
- net /100_CPU/A4: track 0.00 -> 160.1 mm, vias 0 -> 3
- net /100_CPU/A1: track 0.00 -> 160.1 mm, vias 0 -> 1
- net /100_CPU/A2: track 0.00 -> 159.2 mm, vias 0 -> 1
- net /100_CPU/D5: track 0.00 -> 158.7 mm, vias 0 -> 1
- net /100_CPU/D7: track 0.00 -> 152.1 mm, vias 0 -> 1
- net /100_CPU/D1: track 0.00 -> 149.7 mm, vias 0 -> 1
- net +5V: track 100.3 -> 248.8 mm, vias 0 -> 8
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Other:
- board text added: "https://github.com/anjennings"

Commit message: gerbers have been sent
Parts:
- removed the REF** at (262.6, 14.7)
- added D1: 1N4001, Diode_THT:D_DO-41_SOD81_P10.16mm_Horizontal, F.Cu at (259.3, 110.5)
- moved REF** 67.6 mm to (262.9, 15.0)
- moved J00 3.05 mm to (240.8, 112.3)
- moved J301 2.54 mm to (255.3, 119.4)
Connections:
- J00 pad 1: VCC -> Net-(D1-Pad2)
Routing:
- net Net-(D1-Pad2): track 0.00 -> 10.9 mm
- net VCC: track 82.5 -> 84.3 mm
