File: kicad/100_CPU.sch (KiCad schematic (older format))
At the start: 9 parts, among them U100 68008D, U101 74LS07, U102 GAL16V8

Commit message: Generated BOM
Other:
- note added: "This page has been checked\n"
- note removed: "This page has NOT been checked\n"
Changed lines of the file:
@@
 Text HLabel 3000 5550 0    50   Input ~ 0
 AS
-Text Notes 4900 1550 0    50   ~ 0
-This page has NOT been checked\n
+Text Notes 4900 1550 0    50   ~ 10
+This page has been checked\n
 NoConn ~ 10100 3450
 Text HLabel 10100 3550 2    50   BiDi ~ 0
