File: kicad/68k8.sch (KiCad schematic (older format))
At the start: 45 parts

Commit message: updates from a long time ago
Parts:
- removed BUF1: 74LS07, symbol 74xx:74LS07
- removed C? (x2): C, symbol Device:C
- removed unit 1 of NOT1
- removed RN?: R_Network08, Resistor_THT:R_Array_SIP9, symbol Device:R_Network08
- removed SW?: SW_Push, symbol Switch:SW_Push
- removed U?: LM555xM, Package_SO:SOIC-8_3.9x4.9mm_P1.27mm, symbol Timer:LM555xM
Connections:
- net labels removed: PU_2, PU_3, PU_6
- wire segments 245 -> 214
Changed lines of the file:
@@
 $Descr A2 23386 16535
 encoding utf-8
-Sheet 1 2
+Sheet 1 3
 Title "68k8 SBC"
 Date "2021-07-16"
@@
 Text Label 3600 10650 0    50   ~ 0
 A3
-$Comp
-L 74xx:74LS07 BUF1
-U 1 1 614D70EA
-P 20200 12950
-F 0 "BUF1" H 20200 13267 50  0000 C CNN
-F 1 "74LS07" H 20200 13176 50  0000 C CNN
-F 2 "" H 20200 12950 50  0001 C CNN
-F 3 "www.ti.com/lit/ds/symlink/sn74ls07.pdf" H 20200 12950 50  0001 C CNN
-	1    20200 12950
-	1    0    0    -1
-$EndComp
-$Comp
-L 74xx:74LS07 BUF1
-U 2 1 614D7E5F
-P 20200 13600
-F 0 "BUF1" H 20200 13917 50  0000 C CNN
-F 1 "74LS07" H 20200 13826 50  0000 C CNN
-F 2 "" H 20200 13600 50  0001 C CNN
-F 3 "www.ti.com/lit/ds/symlink/sn74ls07.pdf" H 20200 13600 50  0001 C CNN
-	2    20200 13600
-	1    0    0    -1
-$EndComp
-$Comp
-L 74xx:74LS07 BUF1
-U 3 1 614D93B5
-P 20450 14200
-F 0 "BUF1" H 20450 14517 50  0000 C CNN
-F 1 "74LS07" H 20450 14426 50  0000 C CNN
-F 2 "" H 20450 14200 50  0001 C CNN
-F 3 "www.ti.com/lit/ds/symlink/sn74ls07.pdf" H 20450 14200 50  0001 C CNN
-	3    20450 14200
-	1    0    0    -1
-$EndComp
-Wire Wire Line
-	20500 12950 20650 12950
-Wire Wire Line
-	20500 13600 20650 13600
-Wire Wire Line
-	20650 12950 20650 12800
-Wire Wire Line
-	20650 12800 20800 12800
-Text GLabel 20800 12800 2    50   Input ~ 0
-RESET
-Text GLabel 20750 13600 2    50   Input ~ 0
-HALT
-Wire Wire Line
-	20650 13600 20750 13600
-Connection ~ 20650 13600
-$Comp
-L Timer:LM555xM U?
-U 1 1 61569D76
-P 18400 13450
-F 0 "U?" H 18400 14031 50  0000 L TNN
-F 1 "LM555xM" H 18400 13940 50  0000 L TNN
-F 2 "Package_SO:SOIC-8_3.9x4.9mm_P1.27mm" H 19250 13050 50  0001 C CNN
-F 3 "http://www.ti.com/lit/ds/symlink/lm555.pdf" H 19250 13050 50  0001 C CNN
-	1    18400 13450
-	1    0    0    -1
-$EndComp
-$Comp
-L power:GND #PWR?
-U 1 1 6156DCD9
-P 18400 14100
-F 0 "#PWR?" H 18400 13850 50  0001 C CNN
-F 1 "GND" H 18405 13927 50  0000 C CNN
-F 2 "" H 18400 14100 50  0001 C CNN
-F 3 "" H 18400 14100 50  0001 C CNN
-	1    18400 14100
-	1    0    0    -1
-$EndComp
-$Comp
-L Switch:SW_Push SW?
-U 1 1 6156FADE
-P 17300 13250
-F 0 "SW?" H 17300 13535 50  0000 C CNN
-F 1 "SW_Push" H 17300 13444 50  0000 C CNN
-F 2 "" H 17300 13450 50  0001 C CNN
-F 3 "~" H 17300 13450 50  0001 C CNN
-	1    17300 13250
-	1    0    0    -1
-$EndComp
-$Comp
-L power:VCC #PWR?
-U 1 1 6156CD1A
-P 18400 12750
-F 0 "#PWR?" H 18400 12600 50  0001 C CNN
-F 1 "VCC" H 18415 12923 50  0000 C CNN
-F 2 "" H 18400 12750 50  0001 C CNN
-F 3 "" H 18400 12750 50  0001 C CNN
-	1    18400 12750
-	1    0    0    -1
-$EndComp
-$Comp
-L Device:C C?
-U 1 1 61618BC8
-P 17800 13950
-F 0 "C?" H 17915 13996 50  0000 L CNN
-F 1 "C" H 17915 13905 50  0000 L CNN
-F 2 "" H 17838 13800 50  0001 C CNN
-F 3 "~" H 17800 13950 50  0001 C CNN
-	1    17800 13950
-	1    0    0    -1
-$EndComp
-Wire Wire Line
-	18400 13850 18400 14100
-Wire Wire Line
-	17100 14100 17100 13250
-Connection ~ 18400 14100
-Wire Wire Line
-	18900 13250 19300 13250
-Wire Wire Line
-	19300 13250 19300 12950
-Wire Wire Line
-	18900 13450 19300 13450
-Wire Wire Line
-	19300 13450 19300 13250
-Connection ~ 19300 13250
-Wire Wire Line
-	18900 13650 19300 13650
-Wire Wire Line
-	19300 13650 19300 13450
-Connection ~ 19300 13450
-$Comp
-L Device:C C?
-U 1 1 616C0EA1
-P 19300 13950
-F 0 "C?" H 19415 13996 50  0000 L CNN
-F 1 "C" H 19415 13905 50  0000 L CNN
-F 2 "" H 19338 13800 50  0001 C CNN
-F 3 "~" H 19300 13950 50  0001 C CNN
-	1    19300 13950
-	1    0    0    -1
-$EndComp
-Wire Wire Line
-	18400 14100 19300 14100
 Text GLabel 1100 4100 0    50   Input ~ 0
 HALT
@@
 Text GLabel 3750 11150 0    50   Input ~ 0
 RESET
-$Comp
-L 74xx:74LS04 NOT1
-U 1 1 6101E3F3
-P 19600 13250
-F 0 "NOT1" H 19600 13567 50  0000 C CNN
-F 1 "74LS04" H 19600 13476 50  0000 C CNN
-F 2 "" H 19600 13250 50  0001 C CNN
-F 3 "http://www.ti.com/lit/gpn/sn74LS04" H 19600 13250 50  0001 C CNN
-	1    19600 13250
-	1    0    0    -1
-$EndComp
 $Comp
 L 74xx:74LS04 NOT1
@@
 	1    0    0    -1
 $EndComp
-Connection ~ 19300 13650
-Wire Wire Line
-	19300 13650 19300 13800
-Wire Wire Line
-	19900 12950 19900 13250
-Connection ~ 19900 13250
-Wire Wire Line
-	19900 13250 19900 13600
-Connection ~ 17800 14100
-Wire Wire Line
-	17100 14100 17800 14100
-Wire Wire Line
-	17900 13450 17800 13450
-Wire Wire Line
-	17800 13450 17800 13800
-Wire Wire Line
-	17900 13650 17600 13650
-Wire Wire Line
-	17800 14100 18400 14100
-Wire Wire Line
-	20650 13600 20650 13050
-$Comp
-L power:VCC #PWR?
-U 1 1 61522293
-P 21700 12950
-F 0 "#PWR?" H 21700 12800 50  0001 C CNN
-F 1 "VCC" V 21715 13078 50  0000 L CNN
-F 2 "" H 21700 12950 50  0001 C CNN
-F 3 "" H 21700 12950 50  0001 C CNN
-	1    21700 12950
-	0    1    1    0
-$EndComp
-Connection ~ 20650 12950
 $Comp
 L Interface_USB:MCP2221AxP U?
@@
 Wire Wire Line
 	7500 8450 8000 8450
-Text GLabel 21300 13150 0    50   Input ~ 0
-PU_1
 Text GLabel 7900 9550 2    50   Input ~ 0
 PU_1
-Text GLabel 21300 13250 0    50   Input ~ 0
-PU_2
-Text GLabel 21300 13350 0    50   Input ~ 0
-PU_3
-Text GLabel 17850 13100 1    50   Input ~ 0
-PU_2
-Text GLabel 19300 12950 1    50   Input ~ 0
-PU_3
-Wire Wire Line
-	17600 12750 18400 12750
 Wire Wire Line
 	19850 4650 19950 4650
@@
 Text GLabel 10550 11700 2    50   Input ~ 0
 RESET
-$Comp
-L Device:R_Network08 RN?
-U 1 1 61C4E53B
-P 21500 13350
-F 0 "RN?" V 20883 13350 50  0000 C CNN
-F 1 "R_Network08" V 20974 13350 50  0000 C CNN
-F 2 "Resistor_THT:R_Array_SIP9" V 21975 13350 50  0001 C CNN
-F 3 "http://www.vishay.com/docs/31509/csc.pdf" H 21500 13350 50  0001 C CNN
-	1    21500 13350
-	0    1    1    0
-$EndComp
-Wire Wire Line
-	20650 13050 21300 13050
-Wire Wire Line
-	20650 12950 21300 12950
-Text GLabel 21300 13450 0    50   Input ~ 0
-PU_4
-Text GLabel 21300 13550 0    50   Input ~ 0
-PU_5
-Text GLabel 21300 13650 0    50   Input ~ 0
-PU_6
 Text GLabel 900  2000 0    50   Input ~ 0
 MFP_IRQ
@@
 	-1   0    0    1
 $EndComp
-Wire Wire Line
-	17500 13250 17850 13250
-Wire Wire Line
-	17850 13250 17850 13100
-Connection ~ 17850 13250
-Wire Wire Line
-	17850 13250 17900 13250
-Wire Wire Line
-	17600 13650 17600 12750
-Wire Wire Line
-	18400 12750 18400 13050
-Connection ~ 18400 12750
 $Comp
 L 74xx:74LS21 4AND
@@
 Wire Wire Line
 	4950 15700 5350 15700
-Wire Bus Line
-	18100 4700 18100 5000
-Wire Bus Line
-	17400 900  17400 1300
-Wire Bus Line
-	3450 10250 3450 10650
-Wire Bus Line
-	9150 9300 9150 9800
-Wire Bus Line
-	4900 1600 4900 5000
-Wire Bus Line
-	7100 1600 7100 5000
-Wire Bus Line
-	9300 1600 9300 5000
-Wire Bus Line
-	3450 9350 3450 10150
-Wire Bus Line
-	3150 3900 3150 5000
-Wire Bus Line
-	10850 9400 10850 10200
-Wire Bus Line
-	3550 900  3550 2800
-Wire Bus Line
-	7400 900  7400 3200
-Wire Bus Line
-	5200 900  5200 3200
-Wire Bus Line
-	3200 900  3200 3500
 Connection ~ 5350 15700
 Wire Wire Line
@@
 $EndComp
 Connection ~ 4950 15700
+$Sheet
+S 19200 11500 700  650
+U 6110C011
+F0 "Reset_Logic" 50
+F1 "Reset_Logic.sch" 50
+$EndSheet
+Text HLabel 19900 11650 0    50   Input ~ 0
+HALT
+Text HLabel 19900 11750 0    50   Input ~ 0
+RESET
+Text GLabel 19900 11750 2    50   Input ~ 0
+RESET
+Text GLabel 19900 11650 2    50   Input ~ 0
+HALT
+Wire Bus Line
+	18100 4700 18100 5000
+Wire Bus Line
+	17400 900  17400 1300
+Wire Bus Line
+	3450 10250 3450 10650
+Wire Bus Line
+	9150 9300 9150 9800
+Wire Bus Line
+	4900 1600 4900 5000
+Wire Bus Line
+	7100 1600 7100 5000
+Wire Bus Line
+	9300 1600 9300 5000
+Wire Bus Line
+	3450 9350 3450 10150
+Wire Bus Line
+	3150 3900 3150 5000
+Wire Bus Line
+	10850 9400 10850 10200
+Wire Bus Line
+	3550 900  3550 2800
+Wire Bus Line
+	7400 900  7400 3200
+Wire Bus Line
+	5200 900  5200 3200
+Wire Bus Line
+	3200 900  3200 3500
 $EndSCHEMATC

Commit message: Replaced most logic with EEPLD
Parts:
- removed unit 3 of 4AND
- removed 4OR: 4072, symbol 4xxx:4072
- removed unit 4 of AND1
- removed unit 5 of AND1
- removed MFP: MC68901_DIP, symbol 68901_DIP:MC68901_DIP
- removed unit 1 of NAND1
- removed unit 4 of NAND1
- removed unit 5 of NAND1
- removed unit 2 of NOT1
- removed unit 3 of NOT1
- removed unit 4 of NOT1
- removed unit 6 of NOT1
- removed unit 7 of NOT1
- removed NOT2, U? (x5): 74LS04, symbol 74xx:74LS04
- removed OR1, OR2: 74LS32, symbol 74xx:74LS32
- removed unit 2 of OR3
- removed unit 3 of OR3
- removed unit 4 of OR3
- removed unit 5 of OR3
- added BUF? (x3): 74LS07, symbol 74xx:74LS07
- added C? (x2): C, symbol Device:C
- added J?: Micro_SD_Card, symbol Connector:Micro_SD_Card
- added NOT?: 74LS04, symbol 74xx:74LS04
- added RN?: R_Network08, Resistor_THT:R_Array_SIP9, symbol Device:R_Network08
- added SW?: SW_Push, symbol Switch:SW_Push
- added U? (x2): GAL16V8, symbol Logic_Programmable:GAL16V8
- added U?: LM555xM, Package_SO:SOIC-8_3.9x4.9mm_P1.27mm, symbol Timer:LM555xM
Connections:
- net labels added: HRAM_SEL, IO_SEL, LRAM_SEL, MEM_SEL, PU_2, PU_3, PU_6
- net labels removed: DART_SEL, IO1, IO2, IO_ROM, LRAM, MFP_SEL, MICRO_RX, MICRO_TX, RAM_H_SEL, RAM_L_SEL, ROM, nA14, nA15, nA19, nRW
- wire segments 214 -> 229
Other:
- note added: "0x00000 - 0x07FFF ROM (32 K)\n0x08000 - 0x09FFF IO 1 (8K)\n0x0A000 - 0x0BFFF IO 2 (8K)\n0x0C000 - 0x7FFFF Low Ram (464K)\n0x80000 - 0xFFFFF High Ram (512K)\n\nMEM_SEL indicates RAM/ROM\nIO_SEL indicates IO\n\n(Use AS as CLK?)"
- note added: "DS + RW = WRITE\nDS + /RW = READ\n"
- moved on the sheet: C?, CLK, D0, D1, DART, R0, R1, U?, Y?

Commit message: Almost ready to route the PCB fully
Parts:
- removed 4AND: 74LS21, symbol 74xx:74LS21
- removed AND1: 74LS08, symbol 74xx:74LS08
- removed BUF? (x3): 74LS07, symbol 74xx:74LS07
- removed C? (x14): C, symbol Device:C
- removed CLK: CXO_DIP14, Oscillator:Oscillator_DIP-14, symbol Oscillator:CXO_DIP14
- removed CPU: 68008D, symbol CPU_NXP_68000:68008D
- removed D0, D1: LED, symbol Device:LED
- removed DART: 68681, symbol Interface:68681
- removed J?: Micro_SD_Card, symbol Connector:Micro_SD_Card
- removed NAND1: 4011, symbol 4xxx:4011
- removed NOT1, NOT?: 74LS04, symbol 74xx:74LS04
- removed OR3: 74LS32, symbol 74xx:74LS32
- removed R0, R1: 2K, symbol Device:R
- removed RAM_H, RAM_L: AS6C4008-55PCN, Package_DIP:DIP-32_W15.24mm, symbol Memory_RAM:AS6C4008-55PCN
- removed RN?: R_Network08, Resistor_THT:R_Array_SIP9, symbol Device:R_Network08
- removed ROM: 28C256, symbol Memory_EEPROM:28C256
- removed SW?: SW_Push, symbol Switch:SW_Push
- removed U?: MCP2221AxP, Package_DIP:DIP-14_W7.62mm, symbol Interface_USB:MCP2221AxP
- removed U? (x2): GAL16V8, symbol Logic_Programmable:GAL16V8
- removed U?: LM555xM, Package_SO:SOIC-8_3.9x4.9mm_P1.27mm, symbol Timer:LM555xM
- removed Y?: Crystal, symbol Device:Crystal
- added C1: .1uF, Capacitor_THT:CP_Radial_D8.0mm_P2.50mm, symbol Device:C
- added C2: .33uF, Capacitor_THT:CP_Radial_D8.0mm_P2.50mm, symbol Device:C
- added C3: 2.2uF, Capacitor_THT:CP_Radial_D8.0mm_P2.50mm, symbol Device:CP
- added C4: .1uF, Capacitor_THT:CP_Radial_D8.0mm_P2.50mm, symbol Device:CP
- added H0, H1, H2, H3: MountingHole, MountingHole:MountingHole_4mm, symbol Mechanical:MountingHole
- added J0: Barrel_Jack, Connector_BarrelJack:BarrelJack_Horizontal, symbol Connector:Barrel_Jack
- added U1: LF33_TO220, Package_TO_SOT_THT:TO-220-3_Horizontal_TabDown, symbol Regulator_Linear:LF33_TO220
- added U2: L7805, Package_TO_SOT_THT:TO-220-3_Vertical, symbol Regulator_Linear:L7805
Connections:
- net GND: now also C1.2, C2.2, C3.2, C4.2, J0.2, U1.2 (GND), U2.2 (GND)
- net VCC: now also C1.1, C2.1, J0.1, U1.1 (VI), U2.1 (IN)
- new net +3V3: C3.1, U1.3 (VO)
- new net +5V: C4.1, U2.3 (OUT)
- no-connect marks 8 -> 0
Other:
- note added: "This page has NOT been checked\n"
- note removed: "0x00000 - 0x07FFF ROM (32 K)\n0x08000 - 0x09FFF IO 1 (8K)\n0x0A000 - 0x0BFFF IO 2 (8K)\n0x0C000 - 0x7FFFF Low Ram (464K)\n0x80000 - 0xFFFFF High Ram (512K)\n\nMEM_SEL indicates RAM/ROM\nIO_SEL indicates IO\n\n(Use AS as CLK?)"
- note removed: "DS + RW = WRITE\nDS + /RW = READ\n"
- note removed: "Interrupt on here are gonna be tricky\n"
- note removed: "Should be LOW when:\nRom or Ram is selected and INTACK is High\nAn IO Asserts DTACK at any time\n\nINTACK sets Addr to 0xFFFFX so DTACK should not be forced low until the IO agrees"

Commit message: almost done, almost
Parts:
- removed J0: Barrel_Jack, Connector_BarrelJack:BarrelJack_Horizontal, symbol Connector:Barrel_Jack
- added D0: POW_LED, LED_THT:LED_D3.0mm, symbol Device:LED
- added D?: D, symbol Device:D
- added J00: Barrel_Jack_Switch, Connector_BarrelJack:BarrelJack_Horizontal, symbol Connector:Barrel_Jack_Switch
- added R0: 2K, Resistor_THT:R_Axial_DIN0309_L9.0mm_D3.2mm_P2.54mm_Vertical, symbol Device:R
Connections:
- wire segments 14 -> 15
Changed lines of the file:
@@
 FC2
-$Comp
-L Connector:Barrel_Jack J?
-U 1 1 619B3A6D
-P 2150 6200
-AR Path="/619AAD15/619B3A6D" Ref="J?"  Part="1"
-AR Path="/619B3A6D" Ref="J0"  Part="1"
-F 0 "J0" H 2207 6525 50  0000 C CNN
-F 1 "Barrel_Jack" H 2207 6434 50  0000 C CNN
-F 2 "Connector_BarrelJack:BarrelJack_Horizontal" H 2200 6160 50  0001 C CNN
-F 3 "~" H 2200 6160 50  0001 C CNN
-	1    2150 6200
-	1    0    0    -1
-$EndComp
 $Comp
 L Regulator_Linear:L7805 U?
@@
 $EndComp
 Wire Wire Line
-	2450 6100 3600 6100
-Wire Wire Line
 	3600 6100 3600 7000
 Wire Wire Line
@@
 L power:GND #PWR?
 U 1 1 619B3A9C
-P 2450 6300
+P 1450 6300
 AR Path="/619AAD15/619B3A9C" Ref="#PWR?"  Part="1"
 AR Path="/619B3A9C" Ref="#PWR0105"  Part="1"
-F 0 "#PWR0105" H 2450 6050 50  0001 C CNN
-F 1 "GND" H 2455 6127 50  0000 C CNN
-F 2 "" H 2450 6300 50  0001 C CNN
-F 3 "" H 2450 6300 50  0001 C CNN
-	1    2450 6300
+F 0 "#PWR0105" H 1450 6050 50  0001 C CNN
+F 1 "GND" H 1455 6127 50  0000 C CNN
+F 2 "" H 1450 6300 50  0001 C CNN
+F 3 "" H 1450 6300 50  0001 C CNN
+	1    1450 6300
 	1    0    0    -1
 $EndComp
@@
 	1    0    0    -1
 $EndComp
+$Comp
+L Connector:Barrel_Jack_Switch J00
+U 1 1 61AB1FC5
+P 1150 6200
+F 0 "J00" H 1207 6517 50  0000 C CNN
+F 1 "Barrel_Jack_Switch" H 1207 6426 50  0000 C CNN
+F 2 "Connector_BarrelJack:BarrelJack_Horizontal" H 1200 6160 50  0001 C CNN
+F 3 "~" H 1200 6160 50  0001 C CNN
+	1    1150 6200
+	1    0    0    -1
+$EndComp
+Wire Wire Line
+	1450 6200 1450 6300
+Connection ~ 1450 6300
+Wire Wire Line
+	1450 6100 2200 6100
+$Comp
+L Device:LED D0
+U 1 1 61AC5F5F
+P 6250 6650
+F 0 "D0" H 6243 6395 50  0000 C CNN
+F 1 "POW_LED" H 6243 6486 50  0000 C CNN
+F 2 "LED_THT:LED_D3.0mm" H 6250 6650 50  0001 C CNN
+F 3 "~" H 6250 6650 50  0001 C CNN
+	1    6250 6650
+	-1   0    0    1
+$EndComp
+$Comp
+L Device:R R0
+U 1 1 61AC656B
+P 5950 6650
+F 0 "R0" V 6157 6650 50  0000 C CNN
+F 1 "2K" V 6066 6650 50  0000 C CNN
+F 2 "Resistor_THT:R_Axial_DIN0309_L9.0mm_D3.2mm_P2.54mm_Vertical" V 5880 6650 50  0001 C CNN
+F 3 "~" H 5950 6650 50  0001 C CNN
+	1    5950 6650
+	0    -1   -1   0
+$EndComp
+$Comp
+L power:+5V #PWR?
+U 1 1 61AC930C
+P 5800 6650
+AR Path="/619AAD15/61AC930C" Ref="#PWR?"  Part="1"
+AR Path="/61AC930C" Ref="#PWR0151"  Part="1"
+F 0 "#PWR0151" H 5800 6500 50  0001 C CNN
+F 1 "+5V" V 5815 6778 50  0000 L CNN
+F 2 "" H 5800 6650 50  0001 C CNN
+F 3 "" H 5800 6650 50  0001 C CNN
+	1    5800 6650
+	0    -1   -1   0
+$EndComp
+$Comp
+L power:GND #PWR0152
+U 1 1 61AC9631
+P 6400 6650
+F 0 "#PWR0152" H 6400 6400 50  0001 C CNN
+F 1 "GND" V 6405 6522 50  0000 R CNN
+F 2 "" H 6400 6650 50  0001 C CNN
+F 3 "" H 6400 6650 50  0001 C CNN
+	1    6400 6650
+	0    -1   -1   0
+$EndComp
+$Comp
+L Device:D D?
+U 1 1 61AC212B
+P 3450 6100
+F 0 "D?" H 3450 5883 50  0000 C CNN
+F 1 "D" H 3450 5974 50  0000 C CNN
+F 2 "" H 3450 6100 50  0001 C CNN
+F 3 "~" H 3450 6100 50  0001 C CNN
+	1    3450 6100
+	-1   0    0    1
+$EndComp
 $EndSCHEMATC

Commit message: gerbers have been sent
Parts:
- D1: renamed from D?; value D -> 1N4001; footprint (none) -> Diode_THT:D_DO-41_SOD81_P10.16mm_Horizontal
Connections:
- wire segments 15 -> 16
Other:
- moved on the sheet: D1, J00
Changed lines of the file:
@@
 L power:GND #PWR?
 U 1 1 619B3A9C
-P 1450 6300
+P 2550 6300
 AR Path="/619AAD15/619B3A9C" Ref="#PWR?"  Part="1"
 AR Path="/619B3A9C" Ref="#PWR0105"  Part="1"
-F 0 "#PWR0105" H 1450 6050 50  0001 C CNN
-F 1 "GND" H 1455 6127 50  0000 C CNN
-F 2 "" H 1450 6300 50  0001 C CNN
-F 3 "" H 1450 6300 50  0001 C CNN
-	1    1450 6300
+F 0 "#PWR0105" H 2550 6050 50  0001 C CNN
+F 1 "GND" H 2555 6127 50  0000 C CNN
+F 2 "" H 2550 6300 50  0001 C CNN
+F 3 "" H 2550 6300 50  0001 C CNN
+	1    2550 6300
 	1    0    0    -1
 $EndComp
@@
 L Connector:Barrel_Jack_Switch J00
 U 1 1 61AB1FC5
-P 1150 6200
-F 0 "J00" H 1207 6517 50  0000 C CNN
-F 1 "Barrel_Jack_Switch" H 1207 6426 50  0000 C CNN
-F 2 "Connector_BarrelJack:BarrelJack_Horizontal" H 1200 6160 50  0001 C CNN
-F 3 "~" H 1200 6160 50  0001 C CNN
-	1    1150 6200
-	1    0    0    -1
-$EndComp
-Wire Wire Line
-	1450 6200 1450 6300
-Connection ~ 1450 6300
-Wire Wire Line
-	1450 6100 2200 6100
+P 2250 6200
+F 0 "J00" H 2307 6517 50  0000 C CNN
+F 1 "Barrel_Jack_Switch" H 2307 6426 50  0000 C CNN
+F 2 "Connector_BarrelJack:BarrelJack_Horizontal" H 2300 6160 50  0001 C CNN
+F 3 "~" H 2300 6160 50  0001 C CNN
+	1    2250 6200
+	1    0    0    -1
+$EndComp
+Wire Wire Line
+	2550 6200 2550 6300
+Connection ~ 2550 6300
+Wire Wire Line
+	2550 6100 2950 6100
 $Comp
 L Device:LED D0
@@
 $EndComp
 $Comp
-L Device:D D?
+L Device:D D1
 U 1 1 61AC212B
-P 3450 6100
-F 0 "D?" H 3450 5883 50  0000 C CNN
-F 1 "D" H 3450 5974 50  0000 C CNN
-F 2 "" H 3450 6100 50  0001 C CNN
-F 3 "~" H 3450 6100 50  0001 C CNN
-	1    3450 6100
+P 3100 6100
+F 0 "D1" H 3100 5883 50  0000 C CNN
+F 1 "1N4001" H 3100 5974 50  0000 C CNN
+F 2 "Diode_THT:D_DO-41_SOD81_P10.16mm_Horizontal" H 3100 6100 50  0001 C CNN
+F 3 "~" H 3100 6100 50  0001 C CNN
+	1    3100 6100
 	-1   0    0    1
 $EndComp
+Wire Wire Line
+	3250 6100 3600 6100
 $EndSCHEMATC

Commit message: Generated BOM
Other:
- note added: "This page has been checked\n"
- note removed: "This page has NOT been checked\n"
Changed lines of the file:
@@
 Text GLabel 8900 4150 2    50   Output ~ 0
 DTACK
-Text Notes 5150 2400 0    50   ~ 0
-This page has NOT been checked\n
+Text Notes 5150 2400 0    50   ~ 10
+This page has been checked\n
 Text GLabel 3200 4350 2    50   BiDi ~ 0
 RESET_IN
