File: kicad/68k8.sch (KiCad schematic (older format))
At the start: 39 parts

Commit message: Squashed commit of the following:
commit 5bb93159fc2b2eccf3bc7271ff40b3cebe761d34
Author: Aidan Jennings <anjennings@wisc.edu>
Date:   Wed Dec 8 17:37:30 2021 -0600

    more unused files

commit 7e13d52fce64914ddbd187ffc850994f54d80316
Author: Aidan Jennings <anjennings@wisc.edu>
Date:   Wed Dec 8 17:35:57 2021 -0600

    removed duplicates

commit 3c904d8ab7304edb10829b27f2aa829f8b83df97
Author: Aidan Jennings <anjennings@wisc.edu>
Date:   Wed Dec 8 17:34:57 2021 -0600

    Removed unused files

commit 4240c4aeb129f72d8cc0c48be629fdf1716b1885
Author: Aidan Jennings <anjennings@wisc.edu>
Date:   Wed Dec 8 17:28:50 2021 -0600

    Generated BOM

commit 9712eee1581c272787fce02cae0011b0c95c9d8a
Author: Aidan Jennings <anjennings@wisc.edu>
Date:   Sat Dec 4 22:41:30 2021 -0600

    gerbers have been sent

commit 8b869a571c38d07b1c0e9f0503dd143095d2a81c
Author: Aidan Jennings <anjennings@wisc.edu>
Date:   Sat Dec 4 16:39:53 2021 -0600

    almost done, almost

commit 7afaedeb05dbef4147d5279c03851ef0c13e751b
Author: Aidan Jennings <anjennings@wisc.edu>
Date:   Thu Dec 2 21:36:47 2021 -0600

    redid power routes

commit 2547c2d57db4d6f7f0b0a47d1d06db8db576e6e7
Author: Aidan Jennings <anjennings@wisc.edu>
Date:   Wed Dec 1 20:41:20 2021 -0600

    key routes placed

commit e823dbd6b612f23569f377613c2fbd576c15e89a
Author: Aidan Jennings <anjennings@wisc.edu>
Date:   Wed Dec 1 20:32:37 2021 -0600

    redid layout

commit a4b2bb637f3746ada467a8a9dac5a0616812d040
Author: Aidan Jennings <anjennings@wisc.edu>
Date:   Wed Dec 1 19:41:24 2021 -0600

    ran autoroute

commit df892af128dde6eacc008c03aafc18ee9515a01c
Author: Aidan Jennings <anjennings@wisc.edu>
Date:   Tue Nov 30 19:09:02 2021 -0600

    moved larger footprints around a bit

commit 6825348058585d23431bbf306323e68c752b0241
Author: Aidan Jennings <anjennings@wisc.edu>
Date:   Mon Nov 29 20:18:27 2021 -0600

    removed rom/ram routes

commit 7e33bc0b151fd37cb50f832426639da6aec4f1f6
Author: Aidan Jennings <anjenning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
Parts:
- removed 4AND: 74LS21, symbol 74xx:74LS21
- removed 4OR: 4072, symbol 4xxx:4072
- removed AND1: 74LS08, symbol 74xx:74LS08
- removed C? (x12): C, symbol Device:C
- removed CLK: CXO_DIP14, Oscillator:Oscillator_DIP-14, symbol Oscillator:CXO_DIP14
- removed CPU: 68008D, symbol CPU_NXP_68000:68008D
- removed D1: LED, symbol Device:LED
- removed DART: 68681, symbol Interface:68681
- removed MFP: MC68901_DIP, symbol 68901_DIP:MC68901_DIP
- removed NAND1: 4011, symbol 4xxx:4011
- removed NOT1, NOT2, U? (x5): 74LS04, symbol 74xx:74LS04
- removed OR1, OR2, OR3: 74LS32, symbol 74xx:74LS32
- removed R1: 2K, symbol Device:R
- removed RAM_H, RAM_L: AS6C4008-55PCN, Package_DIP:DIP-32_W15.24mm, symbol Memory_RAM:AS6C4008-55PCN
- removed ROM: 28C256, symbol Memory_EEPROM:28C256
- removed U?: MCP2221AxP, Package_DIP:DIP-14_W7.62mm, symbol Interface_USB:MCP2221AxP
- removed Y?: Crystal, symbol Device:Crystal
- added C1: .1uF, Capacitor_THT:CP_Radial_D8.0mm_P2.50mm, symbol Device:C
- added C2: .33uF, Capacitor_THT:CP_Radial_D8.0mm_P2.50mm, symbol Device:C
- added C3: 2.2uF, Capacitor_THT:CP_Radial_D8.0mm_P2.50mm, symbol Device:CP
- added C4: .1uF, Capacitor_THT:CP_Radial_D8.0mm_P2.50mm, symbol Device:CP
- added D1: 1N4001, Diode_THT:D_DO-41_SOD81_P10.16mm_Horizontal, symbol Device:D
- added H0, H1, H2, H3: MountingHole, MountingHole:MountingHole_4mm, symbol Mechanical:MountingHole
- added J00: Barrel_Jack_Switch, Connector_BarrelJack:BarrelJack_Horizontal, symbol Connector:Barrel_Jack_Switch
- added U1: LF33_TO220, Package_TO_SOT_THT:TO-220-3_Horizontal_TabDown, symbol Regulator_Linear:LF33_TO220
- added U2: L7805, Package_TO_SOT_THT:TO-220-3_Vertical, symbol Regulator_Linear:L7805
- D0: value LED -> POW_LED; footprint (none) -> LED_THT:LED_D3.0mm
- R0: footprint (none) -> Resistor_THT:R_Axial_DIN0309_L9.0mm_D3.2mm_P2.54mm_Vertical
Connections:
- net GND: now also D0.1 (K), C1.2, C2.2, C3.2, C4.2, J00.2, J00.3, U1.2 (GND), U2.2 (GND); no longer R0.1
- net VCC: now also C1.1, C2.1, D1.1 (K), U1.1 (VI), U2.1 (IN)
- net at D0.2 (A): now also R0.2
- new net: D1.2 (A), J00.1
- new net +3V3: C3.1, U1.3 (VO)
- new net +5V: C4.1, R0.1, U2.3 (OUT)
- no-connect marks 8 -> 0
Other:
- note added: "This page has been checked\n"
- note removed: "Interrupt on here are gonna be tricky\n"
- note removed: "Should be LOW when:\nRom or Ram is selected and INTACK is High\nAn IO Asserts DTACK at any time\n\nINTACK sets Addr to 0xFFFFX so DTACK should not be forced low until the IO agrees"
